Commit message: right openarm

File: biarm_model/openarm_right.urdf (robot description, URDF)
Before this commit: robot openarm, 14 links, 13 joints
Links:
- removed link openarm_link0
- removed link openarm_link1
- removed link openarm_link2
- removed link openarm_link3
- removed link openarm_link4
- removed link openarm_link5
- removed link openarm_link6
- removed link openarm_link7
- added link openarm_right_link0, mass 1.1432284943239561; collision mesh filename=package://openarm_description/meshes/arm/v10/collision/link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 scale=0.001 0.001 0.001; visual mesh filename=package://openarm_description/meshes/arm/v10/visual/link0.d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 scale=0.001 0.001 0.001
- added link openarm_right_link1, mass 1.1416684646202298; collision mesh filename=package://openarm_description/meshes/arm/v10/collision/link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 scale=0.001 0.001 0.001; visual mesh filename=package://openarm_description/meshes/arm/v10/visual/link1.d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 scale=0.001 0.001 0.001
- added link openarm_right_link2, mass 0.2775092746011571; collision mesh filename=package://openarm_description/meshes/arm/v10/collision/link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 scale=0.001 0.001 0.001; visual mesh filename=package://openarm_description/meshes/arm/v10/visual/link2.d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 scale=0.001 0.001 0.001
- added link openarm_right_link3, mass 1.073863338202347; collision mesh filename=package://openarm_description/meshes/arm/v10/collision/link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 scale=0.001 0.001 0.001; visual mesh filename=package://openarm_description/meshes/arm/v10/visual/link3.d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 scale=0.001 0.001 0.001
- added link openarm_right_link4, mass 0.6348534566833373; collision mesh filename=package://openarm_description/meshes/arm/v10/collision/link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 scale=0.001 0.001 0.001; visual mesh filename=package://openarm_description/meshes/arm/v10/visual/link4.d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 scale=0.001 0.001 0.001
- added link openarm_right_link5, mass 0.6156588026168502; collision mesh filename=package://openarm_description/meshes/arm/v10/collision/link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 scale=0.001 0.001 0.001; visual mesh filename=package://openarm_description/meshes/arm/v10/visual/link5.d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 scale=0.001 0.001 0.001
- added link openarm_right_link6, mass 0.475202773187987; collision mesh filename=package://openarm_description/meshes/arm/v10/collision/link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 scale=0.001 0.001 0.001; visual mesh filename=package://openarm_description/meshes/arm/v10/visual/link6.d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 scale=0.001 0.001 0.001
- added link openarm_right_link7, mass 0.4659771327380578; collision mesh filename=package://openarm_description/meshes/arm/v10/collision/link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 scale=0.001 0.001 0.001; visual mesh filename=package://openarm_description/meshes/arm/v10/visual/link7.d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 scale=0.001 0.001 0.001
Joints:
- removed joint openarm_joint1
- removed joint openarm_joint2
- removed joint openarm_joint3
- removed joint openarm_joint4
- removed joint openarm_joint5
- removed joint openarm_joint6
- removed joint openarm_joint7
- added joint openarm_right_joint1: type revolute, parent openarm_right_link0, child openarm_right_link1, origin xyz=0.0 0.0 0.0625 rpy=0 0 0, axis 0 0 1, limit lower=-1.396263 upper=3.490659 effort=40 velocity=16.754666
- added joint openarm_right_joint2: type revolute, parent openarm_right_link1, child openarm_right_link2, origin xyz=-0.0301 0.0 0.06 rpy=1.57079632679 0 0, axis -1 0 0, limit lower=-0.17453267320510335 upper=3.3161253267948965 effort=40 velocity=16.754666
- added joint openarm_right_joint3: type revolute, parent openarm_right_link2, child openarm_right_link3, origin xyz=0.0301 0.0 0.06625 rpy=0 0 0, axis 0 0 1, limit lower=-1.570796 upper=1.570796 effort=27 velocity=5.445426
- added joint openarm_right_joint4: type revolute, parent openarm_right_link3, child openarm_right_link4, origin xyz=-0.0 0.0315 0.15375 rpy=0 0 0, axis 0 1 0, limit lower=0.0 upper=2.443461 effort=27 velocity=5.445426
- added joint openarm_right_joint5: type revolute, parent openarm_right_link4, child openarm_right_link5, origin xyz=0.0 -0.0315 0.0955 rpy=0 0 0, axis 0 0 1, limit lower=-1.570796 upper=1.570796 effort=7 velocity=20.943946
- added joint openarm_right_joint6: type revolute, parent openarm_right_link5, child openarm_right_link6, origin xyz=0.0375 0.0 0.1205 rpy=0 0 0, axis 1 0 0, limit lower=-0.785398 upper=0.785398 effort=7 velocity=20.943946
- added joint openarm_right_joint7: type revolute, parent openarm_right_link6, child openarm_right_link7, origin xyz=-0.0375 0.0 0.0 rpy=0 0 0, axis 0 1 0, limit lower=-1.570796 upper=1.570796 effort=7 velocity=20.943946
- joint openarm_right_openarm_body_link0_joint: child openarm_link0 -> openarm_right_link0
- joint right_openarm_hand_joint: parent openarm_link7 -> openarm_right_link7
